Commit message: added exra wheels on robot model

File: src/my_robot/urdf/my_robot.xacro (robot description, xacro)
@@ -55,3 +55,47 @@
     </visual>
   </link>
+  <link name="Left_wheel">
+    <origin xyz="0 0 0" rpy="0 1.5707 1.5707"/>
+      <inertial>
+      <mass value="5.0"/>
+      <origin xyz="0.0 0 0" rpy=" 0 0 0"/>
+      <inertia
+          ixx="0.1" ixy="0" ixz="0"
+          iyy="0.1" iyz="0"
+          izz="0.1"
+               />
+     </inertial>
+    <geometry>
+      <cylinder radius="0.1" length=".05"/>
+    </geometry>
+   <link name="Right_wheel">
+    <origin xyz="0 0 0" rpy="0 1.5707 1.5707"/>
+      <inertial>
+      <mass value="5.0"/>
+      <origin xyz="0.0 0 0" rpy=" 0 0 0"/>
+      <inertia
+          ixx="0.1" ixy="0" ixz="0"
+          iyy="0.1" iyz="0"
+          izz="0.1"
+               />
+     </inertial>
+    <geometry>
+      <cylinder radius="0.1" length=".05"/>
+    </geometry>
+   <joint type="continuous" name="left_wheel_hinge">
+    <origin xyz="0 0.15 0" rpy="0 0 0"/>
+    <child link="left_wheel"/>
+    <parent link="chassis"/>
+    <axis xyz="0 1 0" rpy="0 0 0"/>
+    <limit effort="10000" velocity="1000"/>
+    <dynamics damping="1.0" friction="1.0"/>
+  </joint>
+   <joint type="continuous" name="right_wheel_hinge">
+    <origin xyz="0 -0.15 0" rpy="0 0 0"/>
+    <child link="right_wheel"/>
+    <parent link="chassis"/>
+    <axis xyz="0 1 0" rpy="0 0 0"/>
+    <limit effort="10000" velocity="1000"/>
+    <dynamics damping="1.0" friction="1.0"/>
+  </joint>
 </robot>

Commit message: added wheels

File: src/my_robot/urdf/my_robot.xacro (robot description, xacro)
@@ -59,5 +59,5 @@
       <inertial>
       <mass value="5.0"/>
-      <origin xyz="0.0 0 0" rpy=" 0 0 0"/>
+      <origin xyz="0.0 0 0" rpy=" 0 1.5707 1.5707"/>
       <inertia
           ixx="0.1" ixy="0" ixz="0"
@@ -69,4 +69,17 @@
       <cylinder radius="0.1" length=".05"/>
     </geometry>
+     <collision name='collision_left_wheel'>
+      <origin xyz="0 0 0" rpy=" 0 1.5707 1.5707"/>
+      <geometry>
+        <cylinder radius="0.1" length=".05"/>
+      </geometry>
+    </collision>
+    <visual name='left_wheel_visual'>
+      <origin xyz="0 0 0" rpy=" 0 1.5707 1.5707"/>
+      <geometry>
+        <cylinder radius="0.1" length=".05"/>
+      </geometry>
+    </visual>
+   </link>
    <link name="Right_wheel">
     <origin xyz="0 0 0" rpy="0 1.5707 1.5707"/>
@@ -83,7 +96,20 @@
       <cylinder radius="0.1" length=".05"/>
     </geometry>
+     <collision name='collision_right_wheel'>
+      <origin xyz="0 0 0" rpy=" 0 1.5707 1.5707"/>
+      <geometry>
+        <cylinder radius="0.1" length=".05"/>
+      </geometry>
+    </collision>
+    <visual name='left_right_visual'>
+      <origin xyz="0 0 0" rpy=" 0 1.5707 1.5707"/>
+      <geometry>
+        <cylinder radius="0.1" length=".05"/>
+      </geometry>
+    </visual>
+  </link>
    <joint type="continuous" name="left_wheel_hinge">
     <origin xyz="0 0.15 0" rpy="0 0 0"/>
-    <child link="left_wheel"/>
+    <child link="Left_wheel"/>
     <parent link="chassis"/>
     <axis xyz="0 1 0" rpy="0 0 0"/>
@@ -93,5 +119,5 @@
    <joint type="continuous" name="right_wheel_hinge">
     <origin xyz="0 -0.15 0" rpy="0 0 0"/>
-    <child link="right_wheel"/>
+    <child link="Right_wheel"/>
     <parent link="chassis"/>
     <axis xyz="0 1 0" rpy="0 0 0"/>

Commit message: added camera and a joint

File: src/my_robot/urdf/my_robot.xacro (robot description, xacro)
@@ -125,3 +125,34 @@
     <dynamics damping="1.0" friction="1.0"/>
   </joint>
+   <link name='camera'>
+    <pose>0 0 0 0 0 0</pose>
+    <inertial>
+      <mass value=".10"/>
+      <origin xyz="0.0 0 0" rpy=" 0 0 0"/>
+      <inertia
+          ixx="1e-6" ixy="0" ixz="0"
+          iyy="1e-6" iyz="0"
+          izz="1e-6"
+      />
+    </inertial>
+    <collision name='camera_collision'>
+      <origin xyz="0 0 0" rpy=" 0 0 0"/>
+      <geometry>
+        <box size=".05 .05 .05"/>
+      </geometry>
+    </collision>
+    <visual name='camera_visual'>
+      <origin xyz="0 0 0" rpy=" 0 0 0"/>
+      <geometry>
+        <box size=".05 .05 .05"/>
+      </geometry>
+    </visual>
+     <box_inertia m="0.1" x="0.05" y="0.05" z="0.05"/>
+  </link>
+   <joint type="fixed" name="camera_joint">
+    <origin xyz="0.2 0 0" rpy="0 0 0"/>
+    <child link="camera"/>
+    <parent link="chassis"/>
+    <axis xyz="0 1 0" rpy="0 0 0"/>
+  </joint>
 </robot>

Commit message: added lidar to robot model

File: src/my_robot/urdf/my_robot.xacro (robot description, xacro)
@@ -156,3 +156,33 @@
     <axis xyz="0 1 0" rpy="0 0 0"/>
   </joint>
+     <link name='hokuyo'>
+    <pose>0 0 0 0 0 0</pose>
+    <inertial>
+      <mass value="1e-5"/>
+      <origin xyz="0.0 0 0" rpy=" 0 0 0"/>
+      <inertia
+          ixx="1e-6" ixy="0" ixz="0"
+          iyy="1e-6" iyz="0"
+          izz="1e-6"
+      />
+    </inertial>
+    <collision name='hokuyo_collision'>
+      <origin xyz="0 0 0" rpy=" 0 0 0"/>
+      <geometry>
+        <box size=".1 .1 .1"/>
+      </geometry>
+    </collision>
+    <visual name='hokuyo_visual'>
+      <origin xyz="0 0 0" rpy=" 0 0 0"/>
+      <geometry>
+        <filename="package://my_robot/meshes/hokuyo.dae"/>
+      </geometry>
+    </visual>
+  </link>
+   <joint type="fixed" name="hokuyo_joint">
+    <origin xyz="0.15 0 .1" rpy="0 0 0"/>
+    <child link="hokuyo"/>
+    <parent link="chassis"/>
+    <axis xyz="0 1 0" rpy="0 0 0"/>
+  </joint>
 </robot>

Commit message: Update my_robot.xacro

File: src/my_robot/urdf/my_robot.xacro (robot description, xacro)
@@ -176,5 +176,5 @@
       <origin xyz="0 0 0" rpy=" 0 0 0"/>
       <geometry>
-        <filename="package://my_robot/meshes/hokuyo.dae"/>
+        <mesh filename="package://my_robot/meshes/hokuyo.dae"/>
       </geometry>
     </visual>

Commit message: Update my_robot.xacro

File: src/my_robot/urdf/my_robot.xacro (robot description, xacro)
@@ -181,5 +181,5 @@
   </link>
    <joint type="fixed" name="hokuyo_joint">
-    <origin xyz="0.15 0 .1" rpy="0 0 0"/>
+    <origin xyz="0.15 0 .01" rpy="0 0 0"/>
     <child link="hokuyo"/>
     <parent link="chassis"/>

Commit message: Update my_robot.xacro

File: src/my_robot/urdf/my_robot.xacro (robot description, xacro)
@@ -181,5 +181,5 @@
   </link>
    <joint type="fixed" name="hokuyo_joint">
-    <origin xyz="0.15 0 .01" rpy="0 0 0"/>
+    <origin xyz="0.15 0 .1" rpy="0 0 0"/>
     <child link="hokuyo"/>
     <parent link="chassis"/>

Commit message: Update my_robot.xacro

File: src/my_robot/urdf/my_robot.xacro (robot description, xacro)
@@ -174,5 +174,5 @@
     </collision>
     <visual name='hokuyo_visual'>
-      <origin xyz="0 0 0" rpy=" 0 0 0"/>
+      <origin xyz="0.15 0 .1" rpy=" 0 0 0"/>
       <geometry>
         <mesh filename="package://my_robot/meshes/hokuyo.dae"/>

Commit message: Update my_robot.xacro

File: src/my_robot/urdf/my_robot.xacro (robot description, xacro)
@@ -174,5 +174,5 @@
     </collision>
     <visual name='hokuyo_visual'>
-      <origin xyz="0.15 0 .1" rpy=" 0 0 0"/>
+      <origin xyz="0 0 -.1" rpy=" 0 0 0"/>
       <geometry>
         <mesh filename="package://my_robot/meshes/hokuyo.dae"/>

Commit message: Update my_robot.xacro

File: src/my_robot/urdf/my_robot.xacro (robot description, xacro)
@@ -174,5 +174,5 @@
     </collision>
     <visual name='hokuyo_visual'>
-      <origin xyz="0 0 -.1" rpy=" 0 0 0"/>
+      <origin xyz="0 0 0" rpy=" 0 0 0"/>
       <geometry>
         <mesh filename="package://my_robot/meshes/hokuyo.dae"/>

Commit message: added 4 wheel robot to world

File: src/my_robot/urdf/my_robot.xacro (robot description, xacro)
@@ -1,5 +1,3 @@
-<?xml version='1.0'?>
 <robot name="my_robot" xmlns:xacro="http://www.ros.org/wiki/xacro">
-  <xacro:include filename="$(find my_robot)/urdf/my_robot.gazebo" />
   <link name="robot_footprint"></link>
   <joint name="robot_footprint_joint" type="fixed">
@@ -22,5 +20,5 @@
       <origin xyz="0 0 0" rpy=" 0 0 0"/>
       <geometry>
-        <box size=".4 .2 .1"/>
+        <box size=".5 .33 .1"/>
       </geometry>
     </collision>
@@ -28,103 +26,199 @@
       <origin xyz="0 0 0" rpy=" 0 0 0"/>
       <geometry>
-        <box size=".4 .2 .1"/>
-      </geometry>
-    </visual>
-    <collision name='back_caster_collision'>
-      <origin xyz="-0.15 0 -0.05" rpy=" 0 0 0"/>
-      <geometry>
-        <sphere radius="0.0499"/>
-      </geometry>
-    </collision>
-    <visual name='back_caster_visual'>
-      <origin xyz="-0.15 0 -0.05" rpy=" 0 0 0"/>
-      <geometry>
-        <sphere radius="0.05"/>
-      </geometry>
-    </visual>
-    <collision name='front_caster_collision'>
-      <origin xyz="0.15 0 -0.05" rpy=" 0 0 0"/>
-      <geometry>
-        <sphere radius="0.0499"/>
-      </geometry>
-    </collision>
-    <visual name='front_caster_visual'>
-      <origin xyz="0.15 0 -0.05" rpy=" 0 0 0"/>
-      <geometry>
-        <sphere radius="0.05"/>
+        <box size=".5 .33 .1"/>
       </geometry>
     </visual>
   </link>
-  <link name="Left_wheel">
-    <origin xyz="0 0 0" rpy="0 1.5707 1.5707"/>
-      <inertial>
-      <mass value="5.0"/>
-      <origin xyz="0.0 0 0" rpy=" 0 1.5707 1.5707"/>
-      <inertia
-          ixx="0.1" ixy="0" ixz="0"
-          iyy="0.1" iyz="0"
-          izz="0.1"
-               />
-     </inertial>
-    <geometry>
-      <cylinder radius="0.1" length=".05"/>
-    </geometry>
-     <collision name='collision_left_wheel'>
-      <origin xyz="0 0 0" rpy=" 0 1.5707 1.5707"/>
-      <geometry>
-        <cylinder radius="0.1" length=".05"/>
-      </geometry>
-    </collision>
-    <visual name='left_wheel_visual'>
-      <origin xyz="0 0 0" rpy=" 0 1.5707 1.5707"/>
-      <geometry>
-        <cylinder radius="0.1" length=".05"/>
-      </geometry>
-    </visual>
-   </link>
-   <link name="Right_wheel">
-    <origin xyz="0 0 0" rpy="0 1.5707 1.5707"/>
-      <inertial>
-      <mass value="5.0"/>
-      <origin xyz="0.0 0 0" rpy=" 0 0 0"/>
-      <inertia
-          ixx="0.1" ixy="0" ixz="0"
-          iyy="0.1" iyz="0"
-          izz="0.1"
-               />
-     </inertial>
-    <geometry>
-      <cylinder radius="0.1" length=".05"/>
-    </geometry>
-     <collision name='collision_right_wheel'>
-      <origin xyz="0 0 0" rpy=" 0 1.5707 1.5707"/>
-      <geometry>
-        <cylinder radius="0.1" length=".05"/>
-      </geometry>
-    </collision>
-    <visual name='left_right_visual'>
-      <origin xyz="0 0 0" rpy=" 0 1.5707 1.5707"/>
-      <geometry>
-        <cylinder radius="0.1" length=".05"/>
-      </geometry>
+ <link name ='right_rear_wheel'>
+	<pose>0 0 0 0 0 0</pose>
+	    <inertial>
+	      <mass value="5.0"/>
+	      <origin xyz="0.0 0 0" rpy=" 0 1.5707 1.5707"/>
+	      <inertia
+		  ixx="0.1" ixy="0" ixz="0"
+		  iyy="0.1" iyz="0"
+		  izz="0.1"
+	      />
+	    </inertial>
+	    <collision name='right_rear_collision'>
+	      <origin xyz="0 0 0" rpy=" 0 1.5707 1.5707"/>
+	      <geometry>
+		<cylinder radius='.15' length='0.05'/>
+	      </geometry>
+	    </collision>
+	    <visual name='right_rear_wheel_visual'>
+	      <origin xyz="0 0 0" rpy=" 0 1.5707 1.5707"/>
+	      <geometry>
+		<cylinder radius='.15' length='0.05'/>
+	      </geometry>
+	    </visual>
+</link>
+<joint type="continuous" name="right_rear_wheel_hinge">
+    <origin xyz="-0.2 -0.2 0" rpy="0 0 0"/>
+    <child link="right_rear_wheel"/>
+    <parent link="chassis"/>
+    <axis xyz="0 1 0" rpy="0 0 0"/>
+    <limit effort="10000" velocity="1000"/>
+    <dynamics damping="1.0" friction="1.0"/>
+  </joint>
+<link name ='right_front_wheel'>
+	<pose>0 0 0 0 0 0</pose>
+	    <inertial>
+	      <mass value="5.0"/>
+	      <origin xyz="0.0 0 0" rpy=" 0 1.5707 1.5707"/>
+	      <inertia
+		  ixx="0.1" ixy="0" ixz="0"
+		  iyy="0.1" iyz="0"
+		  izz="0.1"
+	      />
+	    </inertial>
+	    <collision name='right_front_collision'>
+	      <origin xyz="0 0 0" rpy=" 0 1.5707 1.5707"/>
+	      <geometry>
+		<cylinder radius='.15' length='0.05'/>
+	      </geometry>
+	    </collision>
+	    <visual name='right_front_wheel_visual'>
+	      <origin xyz="0 0 0" rpy=" 0 1.5707 1.5707"/>
+	      <geometry>
+		<cylinder radius='.15' length='0.05'/>
+	      </geometry>
+	    </visual>
+</link>
+<joint type="continuous" name="right_front_wheel_hinge">
+    <origin xyz="0.2 -0.2 0" rpy="0 0 0"/>
+    <child link="right_front_wheel"/>
+    <parent link="chassis"/>
+    <axis xyz="0 1 0" rpy="0 0 0"/>
+    <limit effort="10000" velocity="1000"/>
+    <dynamics damping="1.0" friction="1.0"/>
+  </joint>
+<link name ='left_rear_wheel'>
+	<pose>0 0 0 0 0 0</pose>
+	    <inertial>
+	      <mass value="5.0"/>
+	      <origin xyz="0.0 0 0" rpy=" 0 1.5707 1.5707"/>
+	      <inertia
+		  ixx="0.1" ixy="0" ixz="0"
+		  iyy="0.1" iyz="0"
+		  izz="0.1"
+	      />
+	    </inertial>
+	    <collision name='left_rear_collision'>
+	      <origin xyz="0 0 0" rpy=" 0 1.5707 1.5707"/>
+	      <geometry>
+		<cylinder radius='.15' length='0.05'/>
+	      </geometry>
+	    </collision>
+	    <visual name='left_rear_wheel_visual'>
+	      <origin xyz="0 0 0" rpy=" 0 1.5707 1.5707"/>
+	      <geometry>
+		<cylinder radius='.15' length='0.05'/>
+	      </geometry>
+	    </visual>
+</link>
+<joint type="continuous" name="left_rear_wheel_hinge">
+    <origin xyz="-0.2 0.2 0" rpy="0 0 0"/>
+    <child link="left_rear_wheel"/>
+    <parent link="chassis"/>
+    <axis xyz="0 1 0" rpy="0 0 0"/>
+    <limit effort="10000" velocity="1000"/>
+    <dynamics damping="1.0" friction="1.0"/>
+  </joint>
+<link name ='left_front_wheel'>
+	<pose>0 0 0 0 0 0</pose>
+	    <inertial>
+	      <mass value="5.0"/>
+	      <origin xyz="0.0 0 0" rpy=" 0 1.5707 1.5707"/>
+	      <inertia
+		  ixx="0.1" ixy="0" ixz="0"
+		  iyy="0.1" iyz="0"
+		  izz="0.1"
+	      />
+	    </inertial>
+	    <collision name='left_front_collision'>
+	      <origin xyz="0 0 0" rpy=" 0 1.5707 1.5707"/>
+	      <geometry>
+		<cylinder radius='.15' length='0.05'/>
+	      </geometry>
+	    </collision>
+	    <visual name='left_front_wheel_visual'>
+	      <origin xyz="0 0 0" rpy=" 0 1.5707 1.5707"/>
+	      <geometry>
+		<cylinder radius='.15' length='0.05'/>
+	      </geometry>
+	    </visual>
+</link>
+<joint type="continuous" name="left_front_wheel_hinge">
+    <origin xyz="0.2 0.2 0" rpy="0 0 0"/>
+    <child link="left_front_wheel"/>
+    <parent link="chassis"/>
+    <axis xyz="0 1 0" rpy="0 0 0"/>
+    <limit effort="10000" velocity="1000"/>
+    <dynamics damping="1.0" friction="1.0"/>
+  </joint>
+<link name ='sensor_tower'>
+	<pose>0 0 0 0 0 0</pose>
+	    <inertial>
+	      <mass value="5.0"/>
+	      <origin xyz="0.0 0 0" rpy=" 0 0 0"/>
+	      <inertia
+		  ixx="0.1" ixy="0" ixz="0"
+		  iyy="0.1" iyz="0"
+		  izz="0.1"
+	      />
+	    </inertial>
+	    <collision name='sensor_tower_collision'>
+	      <origin xyz="0 0 0" rpy=" 0 0 0"/>
+	      <geometry>
+		<box size='.15 .15 .1'/>
+	      </geometry>
+	    </collision>
+	    <visual name='sensor_tower_visual'>
+	      <origin xyz="0 0 0" rpy=" 0 0 0"/>
+	      <geometry>
+		<box size='.15 .15 .1'/>
+	      </geometry>
+	    </visual>
+</link>
+<joint type="continuous" name="sensor_tower_joint">
+    <origin xyz="0 0 .1" rpy="0 0 0"/>
+    <child link="sensor_tower"/>
+    <parent link="chassis"/>
+    <axis xyz="1 0 0" rpy="0 0 0"/>
+    <limit effort="10000" velocity="1000"/>
+    <dynamics damping="1.0" friction="1.0"/>
+  </joint>
+<link name='hokuyo'>
+<pose>0 0 0 0 0 0</pose>
+<inertial>
+<mass value="1e-5"/>
+<origin xyz="0.0 0 0" rpy=" 0 0 0"/>
+<inertia
+  ixx="1e-6" ixy="0" ixz="0"
+  iyy="1e-6" iyz="0"
+  izz="1e-6"
+/>
+</inertial>
+<collision name='hokuyo_collision'>
+<origin xyz="0 0 0" rpy=" 0 0 0"/>
+<geometry>
+<mesh filename="package://my_robot/meshes/hokuyo.dae"/>
+</geometry>
+</collision>
+<visual name='hokuyo_visual'>
+<origin xyz="0 0 0" rpy=" 0 0 0"/>
+<geometry>
+<mesh filename="package://my_robot/meshes/hokuyo.dae"/>
+</geometry>
     </visual>
   </link>
-   <joint type="continuous" name="left_wheel_hinge">
-    <origin xyz="0 0.15 0" rpy="0 0 0"/>
-    <child link="Left_wheel"/>
-    <parent link="chassis"/>
-    <axis xyz="0 1 0" rpy="0 0 0"/>
-    <limit effort="10000" velocity="1000"/>
-    <dynamics damping="1.0" friction="1.0"/>
-  </joint>
-   <joint type="continuous" name="right_wheel_hinge">
-    <origin xyz="0 -0.15 0" rpy="0 0 0"/>
-    <child link="Right_wheel"/>
-    <parent link="chassis"/>
-    <axis xyz="0 1 0" rpy="0 0 0"/>
-    <limit effort="10000" velocity="1000"/>
-    <dynamics damping="1.0" friction="1.0"/>
-  </joint>
-   <link name='camera'>
+  <joint type="fixed" name="hokuyo_joint">
+    <origin xyz="0 0 .075" rpy="0 0 0"/>
+    <child link="hokuyo"/>
+    <parent link="sensor_tower"/>
+    <axis xyz="1 0 0" rpy="0 0 0"/>
+  </joint>
+ <link name='camera'>
     <pose>0 0 0 0 0 0</pose>
     <inertial>
@@ -152,38 +246,8 @@
   </link>
    <joint type="fixed" name="camera_joint">
-    <origin xyz="0.2 0 0" rpy="0 0 0"/>
+    <origin xyz="0.1 0 .025" rpy="0 0 0"/>
     <child link="camera"/>
-    <parent link="chassis"/>
-    <axis xyz="0 1 0" rpy="0 0 0"/>
-  </joint>
-     <link name='hokuyo'>
-    <pose>0 0 0 0 0 0</pose>
-    <inertial>
-      <mass value="1e-5"/>
-      <origin xyz="0.0 0 0" rpy=" 0 0 0"/>
-      <inertia
-          ixx="1e-6" ixy="0" ixz="0"
-          iyy="1e-6" iyz="0"
-          izz="1e-6"
-      />
-    </inertial>
-    <collision name='hokuyo_collision'>
-      <origin xyz="0 0 0" rpy=" 0 0 0"/>
-      <geometry>
-        <box size=".1 .1 .1"/>
-      </geometry>
-    </collision>
-    <visual name='hokuyo_visual'>
-      <origin xyz="0 0 0" rpy=" 0 0 0"/>
-      <geometry>
-        <mesh filename="package://my_robot/meshes/hokuyo.dae"/>
-      </geometry>
-    </visual>
-  </link>
-   <joint type="fixed" name="hokuyo_joint">
-    <origin xyz="0.15 0 .1" rpy="0 0 0"/>
-    <child link="hokuyo"/>
-    <parent link="chassis"/>
-    <axis xyz="0 1 0" rpy="0 0 0"/>
+    <parent link="sensor_tower"/>
+    <axis xyz="1 0 0" rpy="0 0 0"/>
   </joint>
 </robot>

Commit message: implemented skid motor controller plugin and everythign is working"

File: src/my_robot/urdf/my_robot.xacro (robot description, xacro)
@@ -1,3 +1,5 @@
+<?xml version='1.0'?>
 <robot name="my_robot" xmlns:xacro="http://www.ros.org/wiki/xacro">
+   <xacro:include filename="$(find my_robot)/urdf/my_robot.gazebo" />
   <link name="robot_footprint"></link>
   <joint name="robot_footprint_joint" type="fixed">
@@ -182,6 +184,6 @@
 	    </visual>
 </link>
-<joint type="continuous" name="sensor_tower_joint">
-    <origin xyz="0 0 .1" rpy="0 0 0"/>
+<joint type="fixed" name="sensor_tower_joint">
+    <origin xyz=".06 0 .1" rpy="0 0 0"/>
     <child link="sensor_tower"/>
     <parent link="chassis"/>
